File: hardware/Game_Console.kicad_pcb (KiCad board)
At the start: 2 copper layers, 100 x 70 mm, 18 parts, among them J2 Bat, J3 Conn_02x05_Odd_Even, J4 Conn_01x07, J5 uSD, J6 PCM5102A, SW1 Reset, SW2 SW_Push, SW3 Select, U1 xl63070_back/boost_module, U2 ESP32-S3-WROOM-1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

Commit message: Фікс проблемних місць
Parts:
- added Q1: NMOS, Package_TO_SOT_SMD:SOT-23, B.Cu at (182.7, 104.9)
- renumbered U5 to U3, U3 to U4, U4 to U5
Connections:
- U2 pad 15: unconnected-(U2-IO3-Pad15) -> DISP_EN
- U3 pad 1: GND -> Net-(Q1-D)
Routing:
- net DISP_EN: track 0.00 -> 35.5 mm, vias 0 -> 1
- net DISP_RST: track 47.4 -> 54.1 mm
- net VVAL: track 63.9 -> 68.2 mm
- net +3V3: track 41.7 -> 45.1 mm
- net Net-(Q1-D): track 0.00 -> 2.97 mm
- net OK: track 23.9 -> 25.0 mm
- net GPIO10: track 51.9 -> 52.6 mm
