File: hardware/Game_Console.kicad_sch (KiCad schematic)
At the start: 18 parts, among them J2 Bat, J3 Conn_02x05_Odd_Even, J4 Conn_01x07, J5 uSD, J6 PCM5102A, SW1 Reset, SW2 SW_Push, SW3 Select, U1 xl63070_back/boost_module, U2 ESP32-S3-WROOM-1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

Commit message: Фікс проблемних місць
Parts:
- added Q1: NMOS, Package_TO_SOT_SMD:SOT-23, symbol Simulation_SPICE:NMOS
- renumbered U5 to U3, U3 to U4, U4 to U5
Connections:
- net GND: now also Q1.2 (S); no longer U3.1 (GND)
- net DISP_EN: now reaches U2.15 (IO3)
- net DISP_EN: now also Q1.1 (G)
- new net: Q1.3 (D), U3.1 (GND)
- no-connect marks 15 -> 14
Other:
- moved on the sheet: U3
